Commit message: updated PR2 description

File: mod_srdl/urdf/pr2.urdf (robot description, URDF)
Before this commit: robot pr2, 88 links, 87 joints
Links:
- removed link narrow_stereo_gazebo_l_stereo_camera_frame
- removed link narrow_stereo_gazebo_l_stereo_camera_optical_frame
- removed link narrow_stereo_gazebo_r_stereo_camera_frame
- removed link narrow_stereo_gazebo_r_stereo_camera_optical_frame
- removed link wide_stereo_gazebo_l_stereo_camera_frame
- removed link wide_stereo_gazebo_l_stereo_camera_optical_frame
- removed link wide_stereo_gazebo_r_stereo_camera_frame
- removed link wide_stereo_gazebo_r_stereo_camera_optical_frame
- added link head_mount_kinect_ir_link, mass 0.1; collision sphere radius=0.0005; visual sphere radius=0.0005
- added link head_mount_kinect_ir_optical_frame
- added link head_mount_kinect_rgb_link, mass 0.1; collision sphere radius=0.0005; visual sphere radius=0.0005
- added link head_mount_kinect_rgb_optical_frame
- added link head_mount_link, mass 0.1; collision sphere radius=0.0005; visual mesh filename=package://pr2_description/meshes/sensors/kinect_prosilica_v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 scale=0.001 0.001 0.001
- added link head_mount_prosilica_link, mass 0.1; collision sphere radius=0.0005; visual sphere radius=0.0005
- added link head_mount_prosilica_optical_frame
- added link narrow_stereo_l_stereo_camera_frame, mass 0.01
- added link narrow_stereo_l_stereo_camera_optical_frame
- added link narrow_stereo_r_stereo_camera_frame, mass 0.01
- added link narrow_stereo_r_stereo_camera_optical_frame
- added link wide_stereo_l_stereo_camera_frame, mass 0.01
- added link wide_stereo_l_stereo_camera_optical_frame
- added link wide_stereo_r_stereo_camera_frame, mass 0.01
- added link wide_stereo_r_stereo_camera_optical_frame
Joints:
- removed joint narrow_stereo_gazebo_l_stereo_camera_frame_joint
- removed joint narrow_stereo_gazebo_l_stereo_camera_optical_frame_joint
- removed joint narrow_stereo_gazebo_r_stereo_camera_frame_joint
- removed joint narrow_stereo_gazebo_r_stereo_camera_optical_frame_joint
- removed joint wide_stereo_gazebo_l_stereo_camera_frame_joint
- removed joint wide_stereo_gazebo_l_stereo_camera_optical_frame_joint
- removed joint wide_stereo_gazebo_r_stereo_camera_frame_joint
- removed joint wide_stereo_gazebo_r_stereo_camera_optical_frame_joint
- added joint head_mount_joint: type fixed, parent head_plate_frame, child head_mount_link, origin xyz=-0.138 0 0.091 rpy=0 0 0
- added joint head_mount_kinect_ir_joint: type fixed, parent head_mount_link, child head_mount_kinect_ir_link, origin xyz=-0.032267 0.0125 0.136453 rpy=0 0 0
- added joint head_mount_kinect_ir_optical_frame_joint: type fixed, parent head_mount_kinect_ir_link, child head_mount_kinect_ir_optical_frame, origin xyz=0.0            0.01         0.0 rpy=-1.57079632679 0.0 -1.57079632679
- added joint head_mount_kinect_rgb_joint: type fixed, parent head_mount_kinect_ir_link, child head_mount_kinect_rgb_link, origin xyz=0 -0.03 0 rpy=0 0 0
- added joint head_mount_kinect_rgb_optical_frame_joint: type fixed, parent head_mount_kinect_rgb_link, child head_mount_kinect_rgb_optical_frame, origin xyz=0.0            0.0         0.0 rpy=-1.57079632679 0.0 -1.57079632679
- added joint head_mount_prosilica_joint: type fixed, parent head_mount_link, child head_mount_prosilica_link, origin xyz=-0.046457 0.0125 0.088921 rpy=0 0 0
- added joint head_mount_prosilica_optical_frame_joint: type fixed, parent head_mount_prosilica_link, child head_mount_prosilica_optical_frame, origin xyz=0.0            0.0         0.0 rpy=-1.57079632679 0.0 -1.57079632679
- added joint narrow_stereo_l_stereo_camera_frame_joint: type fixed, parent narrow_stereo_link, child narrow_stereo_l_stereo_camera_frame, origin xyz=0 0 0 rpy=0 0 0
- added joint narrow_stereo_l_stereo_camera_optical_frame_joint: type fixed, parent narrow_stereo_l_stereo_camera_frame, child narrow_stereo_l_stereo_camera_optical_frame, origin xyz=0 0 0 rpy=-1.57079632679 0.0 -1.57079632679
- added joint narrow_stereo_r_stereo_camera_frame_joint: type fixed, parent narrow_stereo_l_stereo_camera_frame, child narrow_stereo_r_stereo_camera_frame, origin xyz=0.0 -0.09 0.0 rpy=0.0 0.0 0.0
- added joint narrow_stereo_r_stereo_camera_optical_frame_joint: type fixed, parent narrow_stereo_r_stereo_camera_frame, child narrow_stereo_r_stereo_camera_optical_frame, origin xyz=0 0 0 rpy=-1.57079632679 0.0 -1.57079632679
- added joint wide_stereo_l_stereo_camera_frame_joint: type fixed, parent wide_stereo_link, child wide_stereo_l_stereo_camera_frame, origin xyz=0 0 0 rpy=0 0 0
- added joint wide_stereo_l_stereo_camera_optical_frame_joint: type fixed, parent wide_stereo_l_stereo_camera_frame, child wide_stereo_l_stereo_camera_optical_frame, origin xyz=0 0 0 rpy=-1.57079632679 0.0 -1.57079632679
- added joint wide_stereo_r_stereo_camera_frame_joint: type fixed, parent wide_stereo_l_stereo_camera_frame, child wide_stereo_r_stereo_camera_frame, origin xyz=0.0 -0.09 0.0 rpy=0.0 0.0 0.0
- added joint wide_stereo_r_stereo_camera_optical_frame_joint: type fixed, parent wide_stereo_r_stereo_camera_frame, child wide_stereo_r_stereo_camera_optical_frame, origin xyz=0 0 0 rpy=-1.57079632679 0.0 -1.57079632679
- joint bl_caster_l_wheel_joint: limit effort=100 velocity=100 -> effort=7 velocity=15
- joint bl_caster_r_wheel_joint: limit effort=100 velocity=100 -> effort=7 velocity=15
- joint bl_caster_rotation_joint: limit effort=100 velocity=100 -> effort=6.5 velocity=10
- joint br_caster_l_wheel_joint: limit effort=100 velocity=100 -> effort=7 velocity=15
- joint br_caster_r_wheel_joint: limit effort=100 velocity=100 -> effort=7 velocity=15
- joint br_caster_rotation_joint: limit effort=100 velocity=100 -> effort=6.5 velocity=10
- joint fl_caster_l_wheel_joint: limit effort=100 velocity=100 -> effort=7 velocity=15
- joint fl_caster_r_wheel_joint: limit effort=100 velocity=100 -> effort=7 velocity=15
- joint fl_caster_rotation_joint: limit effort=100 velocity=100 -> effort=6.5 velocity=10
- joint fr_caster_l_wheel_joint: limit effort=100 velocity=100 -> effort=7 velocity=15
- joint fr_caster_r_wheel_joint: limit effort=100 velocity=100 -> effort=7 velocity=15
- joint fr_caster_rotation_joint: limit effort=100 velocity=100 -> effort=6.5 velocity=10
- joint projector_wg6802418_frame_joint: origin xyz=0.046457 0.110 0.0546 rpy=0 0 0 -> xyz=0 0.110 0.0546 rpy=0 0 0
