Commit message: Further uncommented some tag from PR2 URDF for unit testing.

File: knowrob_srdl/urdf/pr2_for_unit_tests.urdf (robot description, URDF)
Before this commit: robot pr2, 95 links, 94 joints
Links:
- link torso_lift_motor_screw_link: geometry collision box size=0.5 0.7 0.01; visual box size=0.5 0.7 0.01
