Commit message: iiwa urdf

File: urdf/iiwa.urdf (robot description, URDF)
Before this commit: robot kmr_iiwa, 32 links, 31 joints
Links:
- link gripper_finger_left_link: geometry collision mesh filename=package://iai_wsg_50_description/meshes/WSG-FMF.stl scale=0.001 0.001 0.001; visual mesh filename=package://iai_wsg_50_description/meshes/WSG-FMF.dae scale=1.0 1.0 1.0
- link gripper_finger_right_link: geometry collision mesh filename=package://iai_wsg_50_description/meshes/WSG-FMF.stl scale=0.001 0.001 0.001; visual mesh filename=package://iai_wsg_50_description/meshes/WSG-FMF.dae scale=1.0 1.0 1.0
- link gripper_gripper_left_link: geometry collision mesh filename=package://iai_wsg_50_description/meshes/GUIDE_WSG50_110.stl scale=0.001 0.001 0.001; visual mesh filename=package://iai_wsg_50_description/meshes/GUIDE_WSG50_110.dae scale=1.0 1.0 1.0
- link gripper_gripper_right_link: geometry collision mesh filename=package://iai_wsg_50_description/meshes/GUIDE_WSG50_110.stl scale=0.001 0.001 0.001; visual mesh filename=package://iai_wsg_50_description/meshes/GUIDE_WSG50_110.dae scale=1.0 1.0 1.0

Commit message: use dae

File: urdf/iiwa.urdf (robot description, URDF)
Before this commit: robot kmr_iiwa, 32 links, 31 joints
Links:
- link fwk_fwa_050_frame_in: geometry visual mesh filename=package://iai_adapters_description/meshes/fwk_fwa_050_simpl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 scale=1.0 1.0 1.0

Commit message: revert scale

File: urdf/iiwa.urdf (robot description, URDF)
Before this commit: robot kmr_iiwa, 32 links, 31 joints
Links:
- link fwk_fwa_050_frame_in: geometry visual mesh filename=package://iai_adapters_description/meshes/fwk_fwa_050_simpl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 scale=0.001 0.001 0.001
